File: DataLogger/DataLogger.kicad_pcb (KiCad board)
At the start: 2 copper layers, 76 x 69.6 mm, 33 parts, among them J1 UART, J2 SPI, J3 I2C, J4 Battery, J5 Conn_01x06_Pin, J6 Conn_01x04_Pin, SW1 SW_Push, SW2 SW_SPDT, U1 ATmega328-P, U2 24LC1025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

Commit message: edit via
Routing:
- net GND: vias 15 -> 14
Changed lines of the file:
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@@
-	)
-	(via
-		(at 158.2156 91.023)
-		(size 0.6)
-		(drill 0.3)
-		(layers "F.Cu" "B.Cu")
-		(net 2)
 	)
 	(via
